File: hardware/clock/clock.kicad_pcb (KiCad board)
At the start: 2 copper layers, 110 x 60 mm, 46 parts, among them J1 USB-C, J2 POWER SWITCH, J3 PROG, J4 TFT 2.4, Q1 AO3400A, SW1 BOOT, SW2 EN, SW3 WHITE, SW4 BLACK, SW5 EC11, U1 ESP32-S3-WROOM-1, U2 MCP73831, U3 AP2112K-3.3

Commit message: Bobines : vias d'empilement hors des spires ; puissance et horloge régénérées
Les trois vias d'empilement de chaque bobine du quadrant tombaient dans
les bandes de spires des deux autres couches et court-circuitaient la
bobine ; elles sont décalées radialement hors des bandes, reliées par
un tronçon radial, le net tie posé sur le tronçon de la dernière
jonction dans le creux, et les contrôles maison n'exemptent plus que
les deux pastilles du net tie.

Carte puissance et horloge régénérées avec les générateurs corrigés
(DRC KiCad réduit aux nets ouverts et à la sérigraphie), tableaux et
notes mis à jour, rapports de DRC ignorés par git.
Parts:
- added Q2: AO3401A, Package_TO_SOT_SMD:SOT-23, F.Cu at (72.0, 6.52)
- added R15: 56k, Resistor_SMD:R_0603_1608Metric, F.Cu at (13.3, 10.6)
- added R16: 100k, Resistor_SMD:R_0603_1608Metric, F.Cu at (16.2, 10.6)
- added R17: 100k, Resistor_SMD:R_0603_1608Metric, F.Cu at (73.0, 15.8)
- moved H4 33.6 mm to (73.0, 50.5)
- moved R1 18.0 mm to (19.1, 10.6)
- moved C6 12.8 mm to (61.3, 11.4)
- moved R8 12.8 mm to (64.2, 11.4)
- moved R11 12.4 mm to (61.3, 15.8)
- moved R12 12.4 mm to (64.2, 15.8)
- moved R6 8.73 mm to (33.7, 10.6)
- moved C3 8.73 mm to (25.0, 10.6)
- moved C4 8.73 mm to (27.9, 10.6)
- moved C5 8.73 mm to (36.6, 10.6)
- moved R5 8.73 mm to (30.8, 10.6)
- moved R2 8.73 mm to (22.1, 10.6)
- moved C7 5.82 mm to (67.2, 11.4)
- moved C8 5.82 mm to (70.1, 11.4)
- moved R13 5.82 mm to (67.2, 15.8)
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Connections:
- J1 pad A6: USB_DP -> (no net)
- J1 pad A7: USB_DM -> (no net)
- J1 pad A8: SBU1 -> (no net)
- J1 pad B6: USB_DP -> (no net)
- J1 pad B7: USB_DM -> (no net)
- J1 pad B8: SBU2 -> (no net)
- U1 pad 38: LED_CHG -> CHG_SENSE
- U1 pad 7: TFT_LED -> TFT_LED_N
- U3 pad 4: NC -> (no net)
Routing:
- net VBAT_SENSE: track 6.15 -> 125.6 mm, vias 0 -> 1
- net 3V3: track 216.8 -> 101.0 mm
- net CC1: track 0.00 -> 76.7 mm, vias 0 -> 1
- net TFT_LED_N: track 0.00 -> 43.8 mm, vias 0 -> 3
- net VSW: track 135.5 -> 99.9 mm, vias 8 -> 7
- net USB_DP: track 22.0 -> 0.00 mm, vias 1 -> 0
- net BUZZER: track 66.2 -> 79.7 mm, vias 2 -> 1
- net TFT_CS: track 60.1 -> 48.3 mm, vias 2 -> 3
- net ESP_EN: track 108.9 -> 120.1 mm, vias 7 -> 8
- net SBU1: track 9.30 -> 0.00 mm, vias 1 -> 0
- net ENC_A: track 36.9 -> 45.9 mm, vias 4 -> 2
- net VCELL: track 70.3 -> 79.0 mm, vias 5 -> 6
- net CHG_SENSE: track 0.00 -> 8.30 mm, vias 0 -> 1
- net CHG_STAT: track 16.6 -> 24.0 mm
- net PROG: track 10.9 -> 3.70 mm
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