File: hardware/clock/clock.kicad_sch (KiCad schematic)
At the start: 46 parts, among them J1 USB-C, J2 POWER SWITCH, J3 PROG, J4 TFT 2.4, Q1 AO3400A, SW1 BOOT, SW2 EN, SW3 WHITE, SW4 BLACK, SW5 EC11, U1 ESP32-S3-WROOM-1, U2 MCP73831, U3 AP2112K-3.3

Commit message: Bobines : vias d'empilement hors des spires ; puissance et horloge régénérées
Les trois vias d'empilement de chaque bobine du quadrant tombaient dans
les bandes de spires des deux autres couches et court-circuitaient la
bobine ; elles sont décalées radialement hors des bandes, reliées par
un tronçon radial, le net tie posé sur le tronçon de la dernière
jonction dans le creux, et les contrôles maison n'exemptent plus que
les deux pastilles du net tie.

Carte puissance et horloge régénérées avec les générateurs corrigés
(DRC KiCad réduit aux nets ouverts et à la sérigraphie), tableaux et
notes mis à jour, rapports de DRC ignorés par git.
Parts:
- added Q2: AO3401A, Package_TO_SOT_SMD:SOT-23, symbol Transistor_FET:TP0610T
- added R15: 56k, Resistor_SMD:R_0603_1608Metric, symbol Device:R
- added R16, R17: 100k, Resistor_SMD:R_0603_1608Metric, symbol Device:R
Connections:
- net 3V3: now also Q2.2 (S), R17.2
- net CHG_STAT: now also R15.1
- net GND: now also R16.2
- net TFT_LED: now also Q2.3 (D); no longer U1.7 (IO7)
- net LED_CHG renamed CHG_SENSE
- net CHG_SENSE: now also R15.2, R16.1
- net NC: no longer names the net of U3.4 (NC)
- net SBU1: no longer names the net of J1.A8 (SBU1)
- net SBU2: no longer names the net of J1.B8 (SBU2)
- net USB_DM: no longer names the net of J1.A7 (D-)
- net USB_DM: no longer J1.B7 (D-)
- net USB_DP: no longer names the net of J1.A6 (D+)
- net USB_DP: no longer J1.B6 (D+)
- new net TFT_LED_N: Q2.1 (G), R17.1, U1.7 (IO7)
- no-connect marks 17 -> 24
