File: hardware/power/power.kicad_sch (KiCad schematic)
At the start: 82 parts, among them J1 PD 20V IN, J2 POWER SWITCH, J3 BRAIN, J4 CELLS, Q1 AO3400A, Q2 AO3400A, Q3 AO3400A, Q4 AO3400A, Q5 AO3400A, Q6 AO3400A, SW1 WAKE, U1 BQ24610, U2 BQ76920, U3 INA219

Commit message: Bobines : vias d'empilement hors des spires ; puissance et horloge régénérées
Les trois vias d'empilement de chaque bobine du quadrant tombaient dans
les bandes de spires des deux autres couches et court-circuitaient la
bobine ; elles sont décalées radialement hors des bandes, reliées par
un tronçon radial, le net tie posé sur le tronçon de la dernière
jonction dans le creux, et les contrôles maison n'exemptent plus que
les deux pastilles du net tie.

Carte puissance et horloge régénérées avec les générateurs corrigés
(DRC KiCad réduit aux nets ouverts et à la sérigraphie), tableaux et
notes mis à jour, rapports de DRC ignorés par git.
Parts:
- removed Q1, Q2: AO3400A, Package_TO_SOT_SMD:SOT-23, symbol Transistor_FET:BSS138
- removed R16: 0R, Resistor_SMD:R_0603_1608Metric, symbol Device:R
- added Q1, Q2: AO3401A, Package_TO_SOT_SMD:SOT-23, symbol Transistor_FET:TP0610T
- added R39: 30k1, Resistor_SMD:R_0603_1608Metric, symbol Device:R
- R11: value 10k -> 3k16
- R13: value 50k -> 17k8
- R17: value 10m -> 50m
- R7: value 10k -> 5k23
- R9: value 50k -> 43k2
Connections:
- net ACDRV: now also Q1.1 (G), Q2.1 (G)
- net ACMID: now also Q1.3 (D), Q2.3 (D)
- net ACN: now also Q1.2 (S)
- net GND: now also Q6.2 (S), R33.2, R39.2; no longer Q5.2 (S), R32.2
- net PACK-PRE: now also Q5.2 (S), R32.2; no longer Q6.2 (S), R33.2
- net REGN: no longer R7.2
- net TS: now also R7.2, R39.1; no longer R7.1
- net VCHG_IN: now also Q2.2 (S)
- net VREF: now also R7.1
- net AFE_NC: no longer names the net of U2.11 (NC)
- net BATDRV: no longer names the net of U1.23 (~{BATDRV})
- no-connect marks 0 -> 2
