File: hardware/quadrant/quadrant.kicad_pcb (KiCad board)
At the start: 4 copper layers, 220 x 200 mm, 347 parts, among them J1 FPC 16, P1 NPTH, Q1 AO3401A, Q111 AO3400A, Q112 AO3401A, Q121 AO3400A, Q122 AO3401A, Q131 AO3400A, Q132 AO3401A, Q141 AO3400A, Q142 AO3401A, Q151 AO3400A, Q152 AO3401A, Q161 AO3400A, Q162 AO3401A, Q171 AO3400A, Q172 AO3401A, Q181 AO3400A, Q182 AO3401A, Q191 AO3400A, Q192 AO3401A, Q2 AO3400A, Q201 AO3400A, Q202 AO3401A, Q211 AO3400A, Q212 AO3401A, Q221 AO3400A, Q222 AO3401A, Q231 AO3400A, Q232 AO3401A, Q241 AO3400A, Q242 AO3401A, Q251 AO3400A, Q252 AO3401A, Q261 AO3400A, Q262 AO3401A, U1 74HC4514, U2 74HC154, U3 ADG1607, U4 ADG1607, U5 AD8421, U6 74LVC1G04, U7 OPA2810, U8 OPA2810

Commit message: Quadrant : build final (pastilles libres bloquantes, vias fusionnées)
Routing:
- net GND: track 2285.2 -> 2287.2 mm, vias 81 -> 82
Changed lines of the file:
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@@
   (via (at 10.7 29.1) (size 0.6) (drill 0.3) (layers "F.Cu" "B.Cu") (net 35))
   (via (at 2 20.7) (size 0.6) (drill 0.3) (layers "F.Cu" "B.Cu") (net 35))
-  (segment (start 16.3 110.2) (end 16.1 110.2) (width 0.4) (layer "F.Cu") (net 34))
-  (segment (start 16.1 110.2) (end 16.1 110.8) (width 0.4) (layer "F.Cu") (net 34))
   (segment (start 10 7.2) (end 10 7) (width 0.4) (layer "F.Cu") (net 34))
   (segment (start 10 7) (end 10.7 7) (width 0.4) (layer "F.Cu") (net 34))
@@
   (segment (start 4.2 102.5) (end 3.7 102.5) (width 0.4) (layer "F.Cu") (net 34))
   (segment (start 2.8 102.8) (end 2 102.8) (width 0.4) (layer "F.Cu") (net 34))
+  (segment (start 12.8 116.3) (end 13.1 116.3) (width 0.4) (layer "In1.Cu") (net 34))
+  (segment (start 13.1 116.3) (end 13.1 113.8) (width 0.4) (layer "In1.Cu") (net 34))
+  (via (at 13.1 113.8) (size 0.6) (drill 0.3) (layers "F.Cu" "B.Cu") (net 34))
   (segment (start 7.8 106) (end 9.3 106) (width 0.4) (layer "F.Cu") (net 34))
   (segment (start 9.3 106) (end 9.3 109.8) (width 0.4) (layer "F.Cu") (net 34))
