File: hardware/quadrant/quadrant.kicad_sch (KiCad schematic)
At the start: 344 parts, among them J1 FPC 16, Q1 AO3401A, Q111 AO3400A, Q112 AO3401A, Q121 AO3400A, Q122 AO3401A, Q131 AO3400A, Q132 AO3401A, Q141 AO3400A, Q142 AO3401A, Q151 AO3400A, Q152 AO3401A, Q161 AO3400A, Q162 AO3401A, Q171 AO3400A, Q172 AO3401A, Q181 AO3400A, Q182 AO3401A, Q191 AO3400A, Q192 AO3401A, Q2 AO3400A, Q201 AO3400A, Q202 AO3401A, Q211 AO3400A, Q212 AO3401A, Q221 AO3400A, Q222 AO3401A, Q231 AO3400A, Q232 AO3401A, Q241 AO3400A, Q242 AO3401A, Q251 AO3400A, Q252 AO3401A, Q261 AO3400A, Q262 AO3401A, U1 74HC4514, U2 74HC154, U3 ADG1607, U4 ADG1607, U5 AD8421, U6 74LVC1G04, U7 OPA2810, U8 OPA2810

Commit message: Quadrant régénéré avec les bobines corrigées ; pastilles libres bloquantes pour le routeur
Le routeur du frontal ignorait les pastilles non connectées (NC des
mux) et y faisait passer une piste de masse : toute pastille libre est
désormais un obstacle dans le routeur et dans les contrôles. Quadrant
régénéré avec les vias d'empilement décalées et le net tie dans le
creux ; note 14 complétée.
Connections:
- net 5VA: no longer C1.2, C13.2, C16.2, C2.2, C21.2, C22.2, C23.2, C24.2, C3.2, C4.2, C5.2, C6.2, C7.2, C8.2, CL1.2, CL10.2, CL11.2, CL12.2, CL13.2, CL14.2, CL15.2, CL16.2, CL17.2, CL18.2, CL19.2, CL2.2, CL20.2, CL21.2, CL22.2, CL23.2, CL24.2, CL25.2, CL26.2, CL27.2, CL28.2, CL29.2, CL3.2, CL30.2, CL31.2, CL32.2, CL4.2, CL5.2, CL6.2, CL7.2, CL8.2, CL9.2, D111.1 (K), D112.1 (K), D121.1 (K), D122.1 (K), D131.1 (K), D132.1 (K), D141.1 (K), D142.1 (K), D151.1 (K), D152.1 (K), D161.1 (K), D162.1 (K), D171.1 (K), D172.1 (K), D181.1 (K), D182.1 (K), D191.1 (K), D192.1 (K), D201.1 (K), D202.1 (K), D211.1 (K), D212.1 (K), D221.1 (K), D222.1 (K), D231.1 (K), D232.1 (K), D241.1 (K), D242.1 (K), D251.1 (K), D252.1 (K), D261.1 (K), D262.1 (K), D3.1 (K), J1.1 (Pin_1), J1.3 (Pin_3), LD1.3 (VSS), LD10.3 (VSS), LD11.3 (VSS), LD12.3 (VSS), LD13.3 (VSS), LD14.3 (VSS), LD15.3 (VSS), LD16.3 (VSS), LD17.3 (VSS), LD18.3 (VSS), LD19.3 (VSS), LD2.3 (VSS), LD20.3 (VSS), LD21.3 (VSS), LD22.3 (VSS), LD23.3 (VSS), LD24.3 (VSS), LD25.3 (VSS), LD26.3 (VSS), LD27.3 (VSS), LD28.3 (VSS), LD29.3 (VSS), LD3.3 (VSS), LD30.3 (VSS), LD31.3 (VSS), LD32.3 (VSS), LD4.3 (VSS), LD5.3 (VSS), LD6.3 (VSS), LD7.3 (VSS), LD8.3 (VSS), LD9.3 (VSS), Q111.2 (S), Q121.2 (S), Q131.2 (S), Q141.2 (S), Q151.2 (S), Q161.2 (S), Q171.2 (S), Q181.2 (S), Q191.2 (S), Q2.2 (S), Q201.2 (S), Q211.2 (S), Q221.2 (S), Q231.2 (S), Q241.2 (S), Q251.2 (S), Q261.2 (S), R10.2, R115.2, R125.2, R135.2, R145.2, R155.2, R165.2, R175.2, R185.2, R195.2, R205.2, R215.2, R225.2, R235.2, R245.2, R255.2, R265.2, R6.2, R8.2, TP4.1, U1.12 (Vss), U2.12 (GND), U2.18 (E0), U3.25 (V_{SS}), U3.33 (V_{SS}), U3.9 (GND), U4.25 (V_{SS}), U4.33 (V_{SS}), U4.9 (GND), U5.5 (Vs-), U6.3 (GND), U7.4 (V-), U8.4 (V-)
- new net GND: C1.2, C13.2, C16.2, C2.2, C21.2, C22.2, C23.2, C24.2, C3.2, C4.2, C5.2, C6.2, C7.2, C8.2, CL1.2, CL10.2, CL11.2, CL12.2, CL13.2, CL14.2, CL15.2, CL16.2, CL17.2, CL18.2, CL19.2, CL2.2, CL20.2, CL21.2, CL22.2, CL23.2, CL24.2, CL25.2, CL26.2, CL27.2, CL28.2, CL29.2, CL3.2, CL30.2, CL31.2, CL32.2, CL4.2, CL5.2, CL6.2, CL7.2, CL8.2, CL9.2, D111.1 (K), D112.1 (K), D121.1 (K), D122.1 (K), D131.1 (K), D132.1 (K), D141.1 (K), D142.1 (K), D151.1 (K), D152.1 (K), D161.1 (K), D162.1 (K), D171.1 (K), D172.1 (K), D181.1 (K), D182.1 (K), D191.1 (K), D192.1 (K), D201.1 (K), D202.1 (K), D211.1 (K), D212.1 (K), D221.1 (K), D222.1 (K), D231.1 (K), D232.1 (K), D241.1 (K), D242.1 (K), D251.1 (K), D252.1 (K), D261.1 (K), D262.1 (K), D3.1 (K), J1.1 (Pin_1), J1.3 (Pin_3), LD1.3 (VSS), LD10.3 (VSS), LD11.3 (VSS), LD12.3 (VSS), LD13.3 (VSS), LD14.3 (VSS), LD15.3 (VSS), LD16.3 (VSS), LD17.3 (VSS), LD18.3 (VSS), LD19.3 (VSS), LD2.3 (VSS), LD20.3 (VSS), LD21.3 (VSS), LD22.3 (VSS), LD23.3 (VSS), LD24.3 (VSS), LD25.3 (VSS), LD26.3 (VSS), LD27.3 (VSS), LD28.3 (VSS), LD29.3 (VSS), LD3.3 (VSS), LD30.3 (VSS), LD31.3 (VSS), LD32.3 (VSS), LD4.3 (VSS), LD5.3 (VSS), LD6.3 (VSS), LD7.3 (VSS), LD8.3 (VSS), LD9.3 (VSS), Q111.2 (S), Q121.2 (S), Q131.2 (S), Q141.2 (S), Q151.2 (S), Q161.2 (S), Q171.2 (S), Q181.2 (S), Q191.2 (S), Q2.2 (S), Q201.2 (S), Q211.2 (S), Q221.2 (S), Q231.2 (S), Q241.2 (S), Q251.2 (S), Q261.2 (S), R10.2, R115.2, R125.2, R135.2, R145.2, R155.2, R165.2, R175.2, R185.2, R195.2, R205.2, R215.2, R225.2, R235.2, R245.2, R255.2, R265.2, R6.2, R8.2, TP4.1, U1.12 (Vss), U2.12 (GND), U2.18 (E0), U3.25 (V_{SS}), U3.33 (V_{SS}), U3.9 (GND), U4.25 (V_{SS}), U4.33 (V_{SS}), U4.9 (GND), U5.5 (Vs-), U6.3 (GND), U7.4 (V-), U8.4 (V-)

Commit message: Quadrant 4 x 4 régénéré : schéma dessiné à huit feuilles, roue libre, BAV99W, résultats de build et de DRC
hardware/quadrant : feuille racine et feuilles rails, cells-1 à
cells-4, select, chain, leds ; PCB reroutée avec le nouveau plan de
cellule. Build : aucune route LED ou alimentation ouverte, aucun défaut
d'isolement, neuf nets du frontal à finir dans pcbnew (VREF route
désormais) ; DRC KiCad sans erreur hors éléments non connectés. README
du quadrant et tableau de résultats de la note 14 à jour, avec la ligne
du quadrant 2 x 2.
Parts:
- removed C1: 10u/25V, Capacitor_SMD:C_1206_3216Metric, symbol Device:C
- removed C13, C23: 1u, Capacitor_SMD:C_0603_1608Metric, symbol Device:C
- removed C14, C15, C16, C21, C22, C3, C4, C5, C6, C7, C8, CL1, CL10, CL11, CL12, CL13, CL14, CL15, CL16, CL17, CL18, CL19, CL2, CL20, CL21, CL22, CL23, CL24, CL25, CL26, CL27, CL28, CL29, CL3, CL30, CL31, CL32, CL4, CL5, CL6, CL7, CL8, CL9: 100n, Capacitor_SMD:C_0603_1608Metric, symbol Device:C
- removed C17, C18, C24: 1n, Capacitor_SMD:C_0603_1608Metric, symbol Device:C
- removed C19, C20: 330p, Capacitor_SMD:C_0603_1608Metric, symbol Device:C
- removed C2: 10u/10V, Capacitor_SMD:C_1206_3216Metric, symbol Device:C
- removed D111, D112, D121, D122, D131, D132, D141, D142, D151, D152, D161, D162, D171, D172, D181, D182, D191, D192, D201, D202, D211, D212, D221, D222, D231, D232, D241, D242, D251, D252, D261, D262, D3: BAV99, Package_TO_SOT_SMD:SOT-23, symbol Diode:BAV99
- removed D113, D123, D133, D143, D153, D163, D173, D183, D193, D203, D213, D223, D233, D243, D253, D263: B5819W, Diode_SMD:D_SOD-123, symbol Device:D_Schottky
- removed D114, D124, D134, D144, D154, D164, D174, D184, D194, D204, D214, D224, D234, D244, D254, D264: SS34FL, Diode_SMD:D_SOD-123F, symbol Diode:SB120
- removed LD1, LD10, LD11, LD12, LD13, LD14, LD15, LD16, LD17, LD18, LD19, LD2, LD20, LD21, LD22, LD23, LD24, LD25, LD26, LD27, LD28, LD29, LD3, LD30, LD31, LD32, LD4, LD5, LD6, LD7, LD8, LD9: WS2812B, LED_SMD:LED_WS2812B_PLCC4_5.0x5.0mm_P3.2mm, symbol LED:WS2812B
- removed NT1: spirale C1, quadgen:COIL_TIE, symbol Device:NetTie_2
- removed NT10: spirale C10, quadgen:COIL_TIE, symbol Device:NetTie_2
- removed NT11: spirale C11, quadgen:COIL_TIE, symbol Device:NetTie_2
- removed NT12: spirale C12, quadgen:COIL_TIE, symbol Device:NetTie_2
- removed NT13: spirale C13, quadgen:COIL_TIE, symbol Device:NetTie_2
- removed NT14: spirale C14, quadgen:COIL_TIE, symbol Device:NetTie_2
- removed NT15: spirale C15, quadgen:COIL_TIE, symbol Device:NetTie_2
- removed NT16: spirale C16, quadgen:COIL_TIE, symbol Device:NetTie_2
- removed NT2: spirale C2, quadgen:COIL_TIE, symbol Device:NetTie_2
- removed NT3: spirale C3, quadgen:COIL_TIE, symbol Device:NetTie_2
- removed NT4: spirale C4, quadgen:COIL_TIE, symbol Device:NetTie_2
- removed NT5: spirale C5, quadgen:COIL_TIE, symbol Device:NetTie_2
- removed NT6: spirale C6, quadgen:COIL_TIE, symbol Device:NetTie_2
- removed NT7: spirale C7, quadgen:COIL_TIE, symbol Device:NetTie_2
- removed NT8: spirale C8, quadgen:COIL_TIE, symbol Device:NetTie_2
- removed NT9: spirale C9, quadgen:COIL_TIE, symbol Device:NetTie_2
- removed Q1, Q112, Q122, Q132, Q142, Q152, Q162, Q172, Q182, Q192, Q202, Q212, Q222, Q232, Q242, Q252, Q262: AO3401A, Package_TO_SOT_SMD:SOT-23, symbol Transistor_FET:TP0610T
- removed Q111, Q121, Q131, Q141, Q151, Q161, Q171, Q181, Q191, Q2, Q201, Q211, Q221, Q231, Q241, Q251, Q261: AO3400A, Package_TO_SOT_SMD:SOT-23, symbol Transistor_FET:BSS138
- removed R10, R12, R13, R8: 100k, Resistor_SMD:R_0603_1608Metric, symbol Device:R
- removed R111, R112, R121, R122, R131, R132, R141, R142, R151, R152, R161, R162, R171, R172, R181, R182, R191, R192, R201, R202, R211, R212, R221, R222, R231, R232, R241, R242, R251, R252, R261, R262, R6, R7: 10k, Resistor_SMD:R_0603_1608Metric, symbol Device:R
- removed R113, R114, R123, R124, R133, R134, R143, R144, R153, R154, R163, R164, R173, R174, R183, R184, R193, R194, R203, R204, R213, R214, R223, R224, R233, R234, R243, R244, R253, R254, R263, R264: 330R, Resistor_SMD:R_0603_1608Metric, symbol Device:R
- removed R115, R117, R125, R127, R135, R137, R145, R147, R155, R157, R165, R167, R175, R177, R185, R187, R195, R197, R205, R207, R215, R217, R225, R227, R235, R237, R245, R247, R255, R257, R265, R267: 100k, Resistor_SMD:R_0402_1005Metric, symbol Device:R
- removed R116, R126, R136, R146, R156, R166, R176, R186, R196, R206, R216, R226, R236, R246, R256, R266: 680R, Resistor_SMD:R_0805_2012Metric, symbol Device:R
- removed R14: 523R, Resistor_SMD:R_0603_1608Metric, symbol Device:R
- removed R15, R16: 787R, Resistor_SMD:R_0603_1608Metric, symbol Device:R
- removed R17, R21: 590R, Resistor_SMD:R_0603_1608Metric, symbol Device:R
- removed R18, R22, R24: 1k, Resistor_SMD:R_0603_1608Metric, symbol Device:R
- removed R19, R20: 750R, Resistor_SMD:R_0603_1608Metric, symbol Device:R
- removed R23: 3.57k, Resistor_SMD:R_0603_1608Metric, symbol Device:R
- removed R25: 49R9, Resistor_SMD:R_0603_1608Metric, symbol Device:R
- removed R5: 20k5, Resistor_SMD:R_0603_1608Metric, symbol Device:R
- removed R9: 10R, Resistor_SMD:R_2010_5025Metric, symbol Device:R
- removed TP1: AMP_OUT, TestPoint:TestPoint_Pad_1.5x1.5mm, symbol Connector:TestPoint
- removed TP2: VREF, TestPoint:TestPoint_Pad_1.5x1.5mm, symbol Connector:TestPoint
- removed TP3: DRIVE_BUS, TestPoint:TestPoint_Pad_1.5x1.5mm, symbol Connector:TestPoint
- removed TP4: GND, TestPoint:TestPoint_Pad_1.5x1.5mm, symbol Connector:TestPoint
- removed U1: 74HC4514, Package_SO:TSSOP-24_4.4x7.8mm_P0.65mm, symbol 4xxx_IEEE:4514
- removed U2: 74HC154, Package_SO:TSSOP-24_4.4x7.8mm_P0.65mm, symbol 74xx:74LS154
- removed U3, U4: ADG1607, Package_CSP:LFCSP-32-1EP_5x5mm_P0.5mm_EP3.1x3.1mm, symbol Analog_Switch:ADG1607xCP
- removed U5: AD8421, Package_SO:SOIC-8_3.9x4.9mm_P1.27mm, symbol Amplifier_Instrumentation:AD8422ARZ
- removed U6: 74LVC1G04, Package_TO_SOT_SMD:SOT-23-5, symbol 74xGxx:74LVC1G04
- removed U7, U8: OPA2810, Package_SO:SOIC-8_3.9x4.9mm_P1.27mm, symbol Amplifier_Operational:NCS2325D
Connections:
- no-connect marks 14 -> 0
Other:
- added sheet Alimentations, VREF et rail d'impulsion (rails.kicad_sch)
- added sheet Cellules de bobine 1 à 4 (cells-1.kicad_sch)
- added sheet Cellules de bobine 13 à 16 (cells-4.kicad_sch)
- added sheet Cellules de bobine 5 à 8 (cells-2.kicad_sch)
- added sheet Cellules de bobine 9 à 12 (cells-3.kicad_sch)
- added sheet Chaîne d'amplification (chain.kicad_sch)
- added sheet LED de camp (leds.kicad_sch)
- added sheet Sélection : décodeurs et multiplexeurs (select.kicad_sch)
- note added: "Quadrant 4 x 4 : liaison au cerveau (J1) et feuilles par fonction"
- note added: "Étiquettes globales : rails, bus d'adresse et nets partagés entre feuilles ; étiquettes locales : nets internes à une feuille."
- note removed: "AMPLIFIER CHAIN"
- note removed: "CAMP LEDS"
- note removed: "CAMP LEDS, DECOUPLING"
- note removed: "COIL CELL 1"
- note removed: "COIL CELL 10"
- note removed: "COIL CELL 11"
- note removed: "COIL CELL 12"
- note removed: "COIL CELL 13"
- note removed: "COIL CELL 14"
- note removed: "COIL CELL 15"
- note removed: "COIL CELL 16"
- note removed: "COIL CELL 2"
- note removed: "COIL CELL 3"
- note removed: "COIL CELL 4"
- note removed: "COIL CELL 5"
- note removed: "COIL CELL 6"
- note removed: "COIL CELL 7"
- note removed: "COIL CELL 8"
- note removed: "COIL CELL 9"
- note removed: "DECODERS"
- note removed: "LINK AND RAILS"
- note removed: "MUXES"
- note removed: "TEST POINTS"
- title: Damier LC, quadrant 4x4 -> Quadrant 4 x 4
