File: hardware/quadrant-2x2/quadrant-2x2.kicad_pcb (KiCad board)
At the start: 4 copper layers, 120 x 108 mm, 129 parts, among them J1 FPC 16, P1 NPTH, Q1 AO3401A, Q111 AO3400A, Q112 AO3401A, Q121 AO3400A, Q122 AO3401A, Q131 AO3400A, Q132 AO3401A, Q141 AO3400A, Q142 AO3401A, Q2 AO3400A, U1 74HC4514, U2 74HC154, U3 ADG1607, U5 AD8421, U6 74LVC1G04, U7 OPA2810, U8 OPA2810

Commit message: Quadrant 2 x 2 régénéré avec les BAV99W et les résistances 0603
Build : aucune route LED ou alimentation ouverte, aucun défaut
d'isolement, deux nets du frontal à finir dans pcbnew (INA_INM une
pastille, GND trois pastilles) ; DRC KiCad sans erreur hors éléments
non connectés. Rendus du PCB et des feuilles mis à jour.
Parts:
- D111, D112, D121, D122, D131, D132, D141, D142: value BAV99 -> BAV99W; footprint Package_TO_SOT_SMD:SOT-23 -> Package_TO_SOT_SMD:SOT-323_SC-70
- R111, R112, R113, R114, R121, R122, R123, R124, R131, R132, R133, R134, R141, R142, R143, R144: footprint Resistor_SMD:R_0402_1005Metric -> Resistor_SMD:R_0603_1608Metric
- R116, R126, R136, R146: footprint Resistor_SMD:R_0603_1608Metric -> Resistor_SMD:R_0805_2012Metric
- moved R146 3.68 mm to (8.90, 33.1)
- moved R116 3.68 mm to (8.90, 47.9)
- moved R126 3.68 mm to (8.90, 40.5)
- moved R136 3.68 mm to (8.90, 57.5)
- moved R124 1.56 mm to (5.40, 39.6)
- moved R134 1.56 mm to (5.40, 56.6)
- moved R144 1.56 mm to (5.40, 32.2)
- moved R114 1.56 mm to (5.40, 47.0)
- moved D132 1.40 mm to (8.90, 55.2)
- moved D112 1.40 mm to (8.90, 45.5)
- moved D122 1.40 mm to (8.90, 38.1)
- moved D142 1.40 mm to (8.90, 30.7)
- moved R142 1.04 mm to (5.40, 30.6)
- moved R112 1.04 mm to (5.40, 45.4)
- moved R122 1.04 mm to (5.40, 38.0)
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Routing:
- net VREF: track 88.9 -> 150.4 mm, vias 8 -> 10
- net DRIVE_BUS: track 111.1 -> 73.5 mm
- net 5VA: track 92.9 -> 116.5 mm, vias 5 -> 9
- net AMP_OUT: track 111.9 -> 134.7 mm, vias 7 -> 8
- net LP_OUT: track 84.2 -> 94.5 mm, vias 5 -> 6
- net HP_IN: track 79.4 -> 85.1 mm, vias 7 -> 6
- net GND: track 745.0 -> 740.0 mm, vias 30 -> 29
- net C4_B: track 685.3 -> 681.6 mm
- net C2_B: track 676.6 -> 672.9 mm
- net PULSE_RAIL: track 114.2 -> 110.7 mm, vias 3 -> 5
- net HP_OUT: track 72.8 -> 69.7 mm, vias 4 -> 3
- net OUT_STAGE: track 90.9 -> 93.9 mm, vias 5 -> 3
- net LP_IN: track 84.0 -> 86.9 mm, vias 3 -> 2
- net DMP3: track 10.9 -> 8.20 mm, vias 2 -> 0
- net DMP2: track 10.8 -> 8.20 mm, vias 2 -> 0
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