File: hardware/quadrant-2x2/cells-1.kicad_sch (KiCad schematic)
At the start: 56 parts, among them Q111 AO3400A, Q112 AO3401A, Q121 AO3400A, Q122 AO3401A, Q131 AO3400A, Q132 AO3401A, Q141 AO3400A, Q142 AO3401A

Commit message: Quadrant 2 x 2 régénéré avec les BAV99W et les résistances 0603
Build : aucune route LED ou alimentation ouverte, aucun défaut
d'isolement, deux nets du frontal à finir dans pcbnew (INA_INM une
pastille, GND trois pastilles) ; DRC KiCad sans erreur hors éléments
non connectés. Rendus du PCB et des feuilles mis à jour.
Parts:
- D111, D112, D121, D122, D131, D132, D141, D142: value BAV99 -> BAV99W; footprint Package_TO_SOT_SMD:SOT-23 -> Package_TO_SOT_SMD:SOT-323_SC-70; LCSC C2500 -> (none); MPN BAV99 -> BAV99W
- R111, R112, R113, R114, R121, R122, R123, R124, R131, R132, R133, R134, R141, R142, R143, R144: footprint Resistor_SMD:R_0402_1005Metric -> Resistor_SMD:R_0603_1608Metric
- R116, R126, R136, R146: footprint Resistor_SMD:R_0603_1608Metric -> Resistor_SMD:R_0805_2012Metric
