File: hardware/bench/bench.kicad_pcb (KiCad board)
At the start: 2 copper layers, 80 x 56 mm, 43 parts, among them J1 12V, J2 QUADRANT, J3 POWER, J4 ANALOG, J5 DIGITAL 0-7, J6 DIGITAL 8-15, U1 TPS62130, U2 LP2985-5.0, U3 74AHCT1G125

Commit message: Carte de banc fermée : éventail FPC et sorties du buck dessinés dans le générateur, connexité vérifiée au build
Le DRC de KiCad comptait 31 connexions manquantes sur la carte de banc
là où le build de boardgen en annonçait six. Cinq trous dans
tools/boardgen/core.py, corrigés : couloir de sortie des vias
d'éventail réclamé sans cuivre (le build dessine maintenant la piste
du couloir jusqu'à la route), pastilles rondes et roundrect prises
pour des rectangles (cellules d'arrivée et contrôle d'isolement sur la
forme réelle), pastille déclarée atteinte sans preuve (vias comptés,
pastille traversante en un seul groupe, sinon net ouvert), piste de
puissance refusée le long d'une piste d'envol (rejouée fine), seeds
disjoints d'un même net jamais rejoints (chaque seed est une pièce de
cuivre, ceux qui se touchent fusionnent). Le build vérifie désormais
la connexité exacte de chaque net après routage et liste en ouvert
tout net en morceaux ; les chutes de masse choisissent une cellule
que le plan atteint ; les empreintes posées reçoivent des tstamp
uniques (le rapport DRC nommait les mauvais éléments). Nouveaux
outils du cœur : seed_via, plain_fanout, cellules de seeds acquises
comme celles des moignons.

Carte de banc : routes manuelles (hand_routes de boardgen/bench.py),
redessinées et vérifiées à chaque build, éventail du FH12 à seize
broches sur les deux faces (voies ouest et est en face avant, groupe
sud en face arrière sous le connecteur jusqu'à J5), montées de la
bande est vers J4 et TP1, longues liaisons 3V3, 5V_LED et AMP_OUT1
en face avant, VIN en face arrière, barrettes SW et VIN du QFN,
ponts de masse au pad thermique, masses murées de U2 et R4 ; TP1 au
coin sud-est. Résultat : 43 composants, 267 segments, 72 vias, 29
nets fermés, zéro ouvert, zéro défaut d'isolement ; DRC KiCad 7.0.11
zéro erreur, zéro élément non connecté.

Tests : la carte de banc doit sortir fermée (test_bench.py), formes
de pastilles et érosion des chutes de masse (test_boardgen_core.py).
Do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
Parts:
- moved TP1 17.5 mm to (78.5, 40.0)
Routing:
- net 3V3: track 1.75 -> 140.2 mm, vias 1 -> 0
- net VIN: track 52.0 -> 130.4 mm, vias 6 -> 9
- net AMP_OUT1: track 2.45 -> 71.9 mm, vias 1 -> 0
- net MUX_EN_L: track 1.75 -> 60.1 mm, vias 1 -> 0
- net LED_DIN1: track 1.75 -> 28.4 mm, vias 1 -> 2
- net 5V: track 112.8 -> 137.8 mm, vias 7 -> 10
- net 5V_LED: track 107.2 -> 125.3 mm, vias 6 -> 4
- net GND: track 15.9 -> 31.7 mm, vias 32 -> 26
- net SW: track 4.66 -> 18.3 mm, vias 2 -> 3
- net LED_END: track 24.1 -> 11.0 mm, vias 2 -> 0
- net PULSE_EN: track 60.8 -> 73.2 mm, vias 3 -> 1
- net 5VA_LDO: track 7.80 -> 19.6 mm, vias 1 -> 2
- net MUX_EN_H: track 54.8 -> 66.3 mm, vias 2 -> 0
- net MUX_A2: track 29.5 -> 35.5 mm, vias 3 -> 1
- net LDO_BP: track 7.95 -> 12.5 mm
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
Commit message: Comptabilité de connexité partagée entre quadgen et boardgen (tools/quadgen/connect.py)
- Module partagé : cuivre réel des pastilles, cellules de treillis
  dans ce cuivre, pièces d'un net par composante de contact exact
  (pastilles, tronçons d'échappée, bus, seeds, vias), boucle de
  fermeture qui n'admet une pastille atteinte que si une route y finit
  ou qu'un via y tombe, cuivre des couloirs de sortie, contrôle de
  connexité final (plans de masse et îlots compris). Tests unitaires.
- boardgen/core.py branché dessus : route_all, chutes de masse par
  pièce, finish ; la carte de banc régénérée reste fermée (29 nets,
  263 segments, DRC KiCad sans erreur ni élément non connecté).
- quadgen/board.py : pastilles à leur forme réelle, deux treillis
  (large et fin) pour la bande, pièces et boucle partagées, cuivre des
  couloirs, seeds manuels, contrôle de connexité en fin de build,
  titre de sérigraphie tiré du plan (2 x 2 ou 4 x 4). Le quadrant
  2 x 2 n'est pas encore régénéré avec ce routage.
- Note 04 : section sur la comptabilité partagée.
Routing:
- net 5VA: track 48.4 -> 47.5 mm
Changed lines of the file:
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@@
   (via (at 51.1 36.913) (size 0.45) (drill 0.2) (layers "F.Cu" "B.Cu") (net 2))
   (via (at 22.61 21.425) (size 0.45) (drill 0.2) (layers "F.Cu" "B.Cu") (net 2))
-  (segment (start 29.55 13.8) (end 29.7 13.8) (width 0.3) (layer "F.Cu") (net 10))
   (segment (start 25.05 16.8) (end 23.55 16.8) (width 0.3) (layer "F.Cu") (net 9))
   (segment (start 23.55 16.8) (end 23.55 23.85) (width 0.3) (layer "F.Cu") (net 9))
@@
   (segment (start 45.45 44.4) (end 45.45 38.85) (width 0.6) (layer "F.Cu") (net 15))
   (segment (start 45.45 38.85) (end 46.05 38.85) (width 0.6) (layer "F.Cu") (net 15))
-  (segment (start 47.55 38.85) (end 47.55 40.35) (width 0.6) (layer "F.Cu") (net 15))
-  (segment (start 47.55 40.35) (end 53.55 40.35) (width 0.6) (layer "F.Cu") (net 15))
-  (segment (start 53.55 40.35) (end 53.55 36.3) (width 0.6) (layer "F.Cu") (net 15))
+  (segment (start 53.55 46.95) (end 53.55 36.3) (width 0.6) (layer "F.Cu") (net 15))
   (segment (start 53.55 36.3) (end 54.6 36.3) (width 0.6) (layer "F.Cu") (net 15))
   (segment (start 21.15 7.95) (end 19.8 7.95) (width 0.6) (layer "B.Cu") (net 7))
@@
   (segment (start 19.65 13.95) (end 20.4 13.95) (width 0.6) (layer "F.Cu") (net 7))
   (via (at 19.8 7.95) (size 0.8) (drill 0.4) (layers "F.Cu" "B.Cu") (net 7))
-  (segment (start 20.4 14.1) (end 19.8 14.1) (width 0.6) (layer "F.Cu") (net 7))
+  (segment (start 19.8 13.95) (end 19.8 14.1) (width 0.6) (layer "F.Cu") (net 7))
   (segment (start 19.8 14.1) (end 18 14.1) (width 0.6) (layer "B.Cu") (net 7))
   (via (at 19.8 14.1) (size 0.8) (drill 0.4) (layers "F.Cu" "B.Cu") (net 7))
@@
   (segment (start 48.45 30) (end 42.45 30) (width 0.6) (layer "F.Cu") (net 4))
   (segment (start 42.45 30) (end 42.45 29.4) (width 0.6) (layer "F.Cu") (net 4))
-  (segment (start 42.6 28.5) (end 42.6 27.15) (width 0.6) (layer "F.Cu") (net 4))
-  (segment (start 42.6 27.15) (end 44.7 27.15) (width 0.6) (layer "F.Cu") (net 4))
-  (segment (start 44.7 27.15) (end 44.7 26.55) (width 0.6) (layer "F.Cu") (net 4))
+  (segment (start 43.95 30) (end 43.95 26.55) (width 0.6) (layer "F.Cu") (net 4))
+  (segment (start 43.95 26.55) (end 44.7 26.55) (width 0.6) (layer "F.Cu") (net 4))
   (segment (start 44.7 25.5) (end 44.7 22.2) (width 0.6) (layer "F.Cu") (net 4))
   (segment (start 48.45 30) (end 49.2 30) (width 0.6) (layer "F.Cu") (net 4))
