File: hardware/brain/brain.kicad_sch (KiCad schematic)
At the start: 113 parts, among them J1 QUADRANT 1, J10 POWER, J2 QUADRANT 2, J3 QUADRANT 3, J4 QUADRANT 4, J5 USB-C, J6 SWD, J7 ESP PROG, J8 PI ZERO, J9 MOTION, Q1 AO3401A, Q2 AO3400A, Q3 AO3400A, SW1 BOOT, SW2 RESET, SW3 ESP BOOT, SW4 ESP EN, SW5 USER, U1 STM32G474RE, U2 TPS62130, U3 AP2112K-3.3, U4 LP2985-5.0, U5 ESP32-S3-WROOM-1, U6 ADuM1201, U7 AMS1117-3.3, U8 74AHCT1G125, U9 USBLC6-2

Commit message: Cerveau : build intermédiaire (module remonté, vias fusionnées)
Connections:
- net COMM_RXD: now also R17.1; no longer R17.2
- net COMM_TXD: now also R16.2; no longer R16.1
- net ESP_RXD: now also R17.2; no longer R16.2
- net ESP_TXD: now also R16.1; no longer R17.1
- net NRST: no longer J6.6 (Pin_6), J6.8 (Pin_8)
- net 3V3_NC: no longer names the net of U3.4 (NC)
- net SBU1: no longer names the net of J5.A8 (SBU1)
- net SBU2: no longer names the net of J5.B8 (SBU2)
- no-connect marks 40 -> 45
