File: hardware/tag-demo/tag-demo.kicad_pcb (KiCad board)
At the start: 2 copper layers, 100 x 86.5 mm, 155 parts, among them U1 G, U10 P+15pF, U11 P+15pF, U12 P+15pF, U13 P+22pF, U14 P+22pF, U15 P+22pF, U2 G, U3 G, U4 G+10pF, U5 G+10pF, U6 G+10pF, U7 P, U8 P, U9 P

Commit message: Planche d'étiquettes : la valeur de chaque puce nomme la pièce et son disque
NT3H2111 suivi de la variante au lieu de la seule lettre du disque ;
carte, rendu, archive et empreintes regénérés, DRC à zéro.
Parts:
- U1, U2, U3: value G -> NT3H2111 G
- U10, U11, U12: value P+15pF -> NT3H2111 P+15pF
- U13, U14, U15: value P+22pF -> NT3H2111 P+22pF
- U4, U5, U6: value G+10pF -> NT3H2111 G+10pF
- U7, U8, U9: value P -> NT3H2111 P
Changed lines of the file:
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@@
         (effects (font (size 1 1) (thickness 0.15)))
     )
-    (fp_text value "G" (at 0 2.55) (layer "F.Fab")
+    (fp_text value "NT3H2111 G" (at 0 2.55) (layer "F.Fab")
         (effects (font (size 1 1) (thickness 0.15)))
     )
@@
         (effects (font (size 1 1) (thickness 0.15)))
     )
-    (fp_text value "G" (at 0 2.55) (layer "F.Fab")
+    (fp_text value "NT3H2111 G" (at 0 2.55) (layer "F.Fab")
         (effects (font (size 1 1) (thickness 0.15)))
     )
@@
         (effects (font (size 1 1) (thickness 0.15)))
     )
-    (fp_text value "G" (at 0 2.55) (layer "F.Fab")
+    (fp_text value "NT3H2111 G" (at 0 2.55) (layer "F.Fab")
         (effects (font (size 1 1) (thickness 0.15)))
     )
@@
         (effects (font (size 1 1) (thickness 0.15)))
     )
-    (fp_text value "G+10pF" (at 0 2.55) (layer "F.Fab")
+    (fp_text value "NT3H2111 G+10pF" (at 0 2.55) (layer "F.Fab")
         (effects (font (size 1 1) (thickness 0.15)))
     )
@@
         (effects (font (size 1 1) (thickness 0.15)))
     )
-    (fp_text value "G+10pF" (at 0 2.55) (layer "F.Fab")
+    (fp_text value "NT3H2111 G+10pF" (at 0 2.55) (layer "F.Fab")
         (effects (font (size 1 1) (thickness 0.15)))
     )
@@
         (effects (font (size 1 1) (thickness 0.15)))
     )
-    (fp_text value "G+10pF" (at 0 2.55) (layer "F.Fab")
+    (fp_text value "NT3H2111 G+10pF" (at 0 2.55) (layer "F.Fab")
         (effects (font (size 1 1) (thickness 0.15)))
     )
@@
         (effects (font (size 1 1) (thickness 0.15)))
     )
-    (fp_text value "P" (at 0 2.55) (layer "F.Fab")
+    (fp_text value "NT3H2111 P" (at 0 2.55) (layer "F.Fab")
         (effects (font (size 1 1) (thickness 0.15)))
     )
@@
         (effects (font (size 1 1) (thickness 0.15)))
     )
-    (fp_text value "P" (at 0 2.55) (layer "F.Fab")
+    (fp_text value "NT3H2111 P" (at 0 2.55) (layer "F.Fab")
         (effects (font (size 1 1) (thickness 0.15)))
     )
@@
         (effects (font (size 1 1) (thickness 0.15)))
     )
-    (fp_text value "P" (at 0 2.55) (layer "F.Fab")
+    (fp_text value "NT3H2111 P" (at 0 2.55) (layer "F.Fab")
         (effects (font (size 1 1) (thickness 0.15)))
     )
@@
         (effects (font (size 1 1) (thickness 0.15)))
     )
-    (fp_text value "P+15pF" (at 0 2.55) (layer "F.Fab")
+    (fp_text value "NT3H2111 P+15pF" (at 0 2.55) (layer "F.Fab")
         (effects (font (size 1 1) (thickness 0.15)))
     )
@@
         (effects (font (size 1 1) (thickness 0.15)))
     )
-    (fp_text value "P+15pF" (at 0 2.55) (layer "F.Fab")
+    (fp_text value "NT3H2111 P+15pF" (at 0 2.55) (layer "F.Fab")
         (effects (font (size 1 1) (thickness 0.15)))
     )
@@
         (effects (font (size 1 1) (thickness 0.15)))
     )
-    (fp_text value "P+15pF" (at 0 2.55) (layer "F.Fab")
+    (fp_text value "NT3H2111 P+15pF" (at 0 2.55) (layer "F.Fab")
         (effects (font (size 1 1) (thickness 0.15)))
     )
@@
         (effects (font (size 1 1) (thickness 0.15)))
     )
-    (fp_text value "P+22pF" (at 0 2.55) (layer "F.Fab")
+    (fp_text value "NT3H2111 P+22pF" (at 0 2.55) (layer "F.Fab")
         (effects (font (size 1 1) (thickness 0.15)))
     )
@@
         (effects (font (size 1 1) (thickness 0.15)))
     )
-    (fp_text value "P+22pF" (at 0 2.55) (layer "F.Fab")
+    (fp_text value "NT3H2111 P+22pF" (at 0 2.55) (layer "F.Fab")
         (effects (font (size 1 1) (thickness 0.15)))
     )
@@
         (effects (font (size 1 1) (thickness 0.15)))
     )
-    (fp_text value "P+22pF" (at 0 2.55) (layer "F.Fab")
+    (fp_text value "NT3H2111 P+22pF" (at 0 2.55) (layer "F.Fab")
         (effects (font (size 1 1) (thickness 0.15)))
     )
